Commit message: Moveit仿真

File: src/my_arm_description/urdf/control1.urdf (robot description, URDF)
Before this commit: robot control1, 8 links, 7 joints
Links:
- added link link4_coupler
Joints:
- removed joint joint4
- added joint joint4_from_joint2: type revolute, parent link3, child link4_coupler, origin xyz=0.08 0.13856 0.017 rpy=1.5708 0 -2.2789, axis 0 -1 0, limit lower=-6.28318 upper=6.28318 effort=100 velocity=2, mimic joint=joint2 multiplier=1.0 offset=0.0
- added joint joint4_from_joint3: type revolute, parent link4_coupler, child link4, origin xyz=0 0 0 rpy=0 0 0, axis 0 -1 0, limit lower=-6.28318 upper=6.28318 effort=100 velocity=2, mimic joint=joint3 multiplier=-1.0 offset=0.0

Commit message: fix: restore link4 horizontal coupling with updated urdf and moveit config

File: src/my_arm_description/urdf/control1.urdf (robot description, URDF)
Before this commit: robot control1, 9 links, 8 joints
Links:
- link base_link: mass 1.1805 -> 0.111516151376738
- link link1: mass 0.246853952260659 -> 0.517175146455813
- link link2: mass 0.16728 -> 0.167276387211561
- link link4: mass 0.0599680536065194 -> 0.0599680536065182
- link link5: mass 0.0332241251365553 -> 0.0332241251365541
- link link6: mass 0.0349726138954135 -> 0.0349726138954209
- link link7: mass 0.0089679 -> 0.00896787232203793
Joints:
- joint joint1: axis 0 -1 0 -> 0 0 -1; limit lower=-3.14 upper=3.14 effort=100 velocity=1 -> lower=-3.14 upper=3.14 effort=0 velocity=0; origin xyz=0 -0.01 0.056 rpy=1.5708 0 3.1416 -> xyz=0 -0.01 0.12105 rpy=0 0 -1.0472; type continuous -> revolute
- joint joint2: axis 0 0 -1 -> 0 -1 0; limit lower=-3.14 upper=3.14 effort=100 velocity=1 -> lower=0 upper=1.57 effort=0 velocity=0; origin xyz=0.0247 0.052 -0.0125 rpy=1.5708 0 1.5708 -> xyz=-0.0040247 -0.031971 -0.013048 rpy=0 -0.5236 2.618
- joint joint3: limit lower=-3.14 upper=3.14 effort=100 velocity=1 -> lower=0 upper=3.14 effort=0 velocity=0; origin xyz=0.08 0.13856 -0.041 rpy=3.1416 0 -0.70807 -> xyz=0.16 -0.046 0 rpy=-1.5708 -1.3863 3.1416
- joint joint4_from_joint2: axis 0 -1 0 -> 1 0 0; origin xyz=0.08 0.13856 0.017 rpy=1.5708 0 -2.2789 -> xyz=0.079999 0.13856 -0.021 rpy=0.70807 1.5708 0
- joint joint4_from_joint3: axis 0 -1 0 -> 1 0 0
- joint joint5: limit lower=-3.14 upper=3.14 effort=100 velocity=1 -> lower=-3.14 upper=3.14 effort=0 velocity=0; origin xyz=-0.0418 -0.025 -0.015 rpy=0 0 0 -> xyz=0 0.041801 0.015001 rpy=3.1416 0 -1.5708; type revolute -> continuous
- joint joint6: limit lower=-3.14 upper=3.14 effort=100 velocity=1 -> lower=-1.57 upper=1.57 effort=0 velocity=0; origin xyz=0 0.012 0 rpy=-3.1416 0.67749 0 -> xyz=0 0.025 0 rpy=-3.1416 0.67749 0
- joint joint7: limit lower=-3.14 upper=3.14 effort=100 velocity=1 -> lower=-3.14 upper=3.14 effort=0 velocity=0
